Commit message: caster wheel was continuous, now fixed

File: my_rb1_description/urdf/my_rb1_robot.urdf (robot description, URDF)
Before this commit: robot robot, 7 links, 6 joints
Joints:
- joint joint_back_caster: type continuous -> fixed
- joint joint_front_caster: type continuous -> fixed

Commit message: Fixed all the mistakes for re-evaluation

File: my_rb1_description/urdf/my_rb1_robot.urdf (robot description, URDF)
Before this commit: robot robot, 7 links, 6 joints
Links:
- link base_link: mass 21 -> 13
- link left_wheel: mass 1 -> 5; geometry collision cylinder length=0.05 radius=0.025; visual cylinder length=0.05 radius=0.025
- link right_wheel: mass 1 -> 5; geometry collision cylinder length=0.05 radius=0.025; visual cylinder length=0.05 radius=0.025
Joints:
- joint joint_back_caster: origin xyz=0.1 0.0 -0.15 rpy=0 0 0 -> xyz=-0.1 0.0 -0.15 rpy=0 0 0
- joint joint_front_caster: origin xyz=-0.1 0.0 -0.15 rpy=0 0 0 -> xyz=0.1 0.0 -0.15 rpy=0 0 0
- joint joint_left_wheel: origin xyz=0.0 -0.2 -0.15 rpy=0 0 0 -> xyz=0.0 0.2 -0.15 rpy=0 0 0
- joint joint_right_wheel: origin xyz=0.0 0.2 -0.15 rpy=0 0 0 -> xyz=0.0 -0.2 -0.15 rpy=0 0 0
